File: hardware/Estacion_lluviaV2/DS3231.kicad_sch (KiCad schematic)
At the start: 7 parts, among them U4 DS3231M

Commit message: Se agregaron nuevos archivos
Parts:
- removed V1: 3, Battery:Battery_Panasonic_CR2032-HFN_Horizontal_CircularHoles, symbol Simulation_SPICE:VDC
- added BT1: SMTU2032-LF, SMTU2032:BAT_SMTU2032-LF, symbol SMTU2032:SMTU2032-LF
- added D3: 1N4148, Diode_SMD:D_SOD-123, symbol Diode:1N4148
Connections:
- net GND: now also BT1.N
- net at U4.14 (VBAT): now also D3.1 (K)
- new net: BT1.P, D3.2 (A)
